File: _autosave-MXR_EnvelopeFilter.kicad_sch (KiCad schematic)
At the start: 63 parts, among them J4 Conn_01x02, Q1 Q_NMOS_GSD, U1 4066, U2 4069, U3 4069, U4 SE8233X2

Commit message: updates
Parts:
- R7: value 10K -> 10M
Changed lines of the file:
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@@
     (in_bom yes) (on_board yes)
     (property "Reference" "R7" (id 0) (at 400.05 121.92 90))
-    (property "Value" "10K" (id 1) (at 400.05 116.84 90))
+    (property "Value" "10M" (id 1) (at 400.05 116.84 90))
     (property "Footprint" "" (id 2) (at 400.05 117.602 90)
       (effects (font (size 1.27 1.27)) hide)
@@
     )
     (path "/cea3126a-864b-4acc-9d3a-01ef1f105f50"
-      (reference "R7") (unit 1) (value "10K") (footprint "")
+      (reference "R7") (unit 1) (value "10M") (footprint "")
     )
     (path "/00000000-0000-0000-0000-00005a2aacf1"
